Commit message: Your commit message

File: src/my_robot/urdf/myrobot.urdf.xacro (robot description, xacro)
@@ -64,8 +64,8 @@
   </xacro:macro>
     <!--wheel with xacro-->
-  <xacro:wheel name="Right_Wheel_Back" x="0.2" y="0.225" z="0.0" r="1.5708" p="0.0" n="0.0"/>
-  <xacro:wheel name="Left_Wheel_Front" x="-0.2" y="-0.225" z="0.0" r="1.5708" p="0.0" n="0.0"/>
-  <xacro:wheel name="Right_Wheel_Front" x="-0.2" y="0.225" z="0.0" r="1.5708" p="0.0" n="0.0"/>
-  <xacro:wheel name="Left_Wheel_Back" x="0.2" y="-0.225" z="0.0" r="1.5708" p="0.0" n="0.0"/>
+  <xacro:wheel name="Left_Wheel_Front" x="0.2" y="0.225" z="0.0" r="1.5708" p="3.14" n="3.14"/>
+  <xacro:wheel name="Right_Wheel_Back" x="-0.2" y="-0.225" z="0.0" r="1.5708" p="3.14" n="3.14"/>
+  <xacro:wheel name="Left_Wheel_Back" x="-0.2" y="0.225" z="0.0" r="1.5708" p="3.14" n="3.14"/>
+  <xacro:wheel name="Right_Wheel_Front" x="0.2" y="-0.225" z="0.0" r="1.5708" p="3.14" n="3.14"/>
     <!-- Hokuyo_lidar -->
   <link name="hokuyo">
@@ -92,5 +92,5 @@
   </link>
   <joint name="hokuyo_joint" type="fixed">
-    <origin xyz="-0.15 0.0 0.1" rpy="0.0 0.0 3.14"/>
+    <origin xyz="0.15 0.0 0.1" rpy="0.0 0.0 0.0"/>
     <parent link="base_link"/>
     <child link="hokuyo"/>
@@ -118,5 +118,5 @@
   </link>
   <joint name="camera_joint" type="fixed">
-      <origin xyz="-0.33 0.0 0.0" rpy="0.0 0.0 3.14"/>
+      <origin xyz="0.33 0.0 0.0" rpy="0.0 0.0 0.0"/>
       <parent link="base_link"/>
       <child link="camera_link"/>
